Commit message: Add urdf macro that allows specifying passthrough components

File: kuka_rsi_driver/urdf/kuka_rsi_driver.ros2_control.xacro (robot description, xacro)
@@ -17,4 +17,23 @@
     rsi_listen_ip
     rsi_listen_port:=49152
+    ">
+    <xacro:kuka_rsi_driver_control_passthrough
+      name="${name}"
+      prefix="${prefix}"
+      use_mock_hardware="${use_mock_hardware}"
+      initial_positions="${initial_positions}"
+      rsi_listen_ip="${rsi_listen_ip}"
+      rsi_listen_port="${rsi_listen_port}">
+      <empty />
+    </xacro:kuka_rsi_driver_control_passthrough>
+  </xacro:macro>
+  <xacro:macro name="kuka_rsi_driver_control_passthrough" params="
+    name
+    prefix
+    use_mock_hardware:=false
+    initial_positions:=${dict(joint_a1=0.0,joint_a2=0.0,joint_a3=0.0,joint_a4=0.0,joint_a5=0.0,joint_a6=0.0)}
+    rsi_listen_ip
+    rsi_listen_port:=49152
+    **passthrough
     ">
     <ros2_control name="${name}" type="system">
@@ -68,13 +87,5 @@
         </state_interface>
       </gpio>
-      <gpio name="qcs">
-        <param name="rsi_name">QCS</param>
-        <state_interface name="sensor_unlocked">
-          <param name="rsi_name">Sensor_Unlocked</param>
-        </state_interface>
-        <state_interface name="sensor_locked">
-          <param name="rsi_name">Sensor_Locked</param>
-        </state_interface>
-      </gpio>
+      <xacro:insert_block name="passthrough" />
     </ros2_control>
   </xacro:macro>
